Commit message: admittance controller addition

File: ros2_control_demo_description/rrbot_description/ros2_control/external_rrbot_force_torque_sensor.ros2_control.xacro (robot description, xacro)
@@ -1,6 +1,6 @@
 <?xml version="1.0"?>
 <robot xmlns:xacro="http://www.ros.org/wiki/xacro">
-  <xacro:macro name="rrbot_system_with_sensor" params="name prefix use_sim:=^|false use_fake_hardware:=^|true fake_sensor_commands:=^|false slowdown:=2.0">
-    <ros2_control name="${name}" type="system">
+  <xacro:macro name="external_rrbot_force_torque_sensor" params="name prefix use_sim:=^|false use_fake_hardware:=^|true fake_sensor_commands:=^|false">
+    <ros2_control name="${name}" type="sensor">
       <hardware>
         <xacro:if value="${use_fake_hardware}">
@@ -10,30 +10,23 @@
         </xacro:if>
         <xacro:unless value="${use_fake_hardware}">
-          <plugin>ros2_control_demo_hardware/RRBotSystemWithSensorHardware</plugin>
+          <plugin>ros2_control_demo_hardware/ExternalRRBotForceTorqueSensorHardware</plugin>
           <param name="example_param_hw_start_duration_sec">0.0</param>
           <param name="example_param_hw_stop_duration_sec">3.0</param>
-          <param name="example_param_hw_slowdown">${slowdown}</param>
           <param name="example_param_max_sensor_change">5.0</param>
         </xacro:unless>
       </hardware>
-      <joint name="${prefix}joint1">
-        <command_interface name="position">
-          <param name="min">-1</param>
-          <param name="max">1</param>
-        </command_interface>
-        <state_interface name="position"/>
-      </joint>
-      <joint name="${prefix}joint2">
-        <command_interface name="position">
-          <param name="min">-1</param>
-          <param name="max">1</param>
-        </command_interface>
-        <state_interface name="position"/>
-      </joint>
       <sensor name="${prefix}tcp_fts_sensor">
         <state_interface name="force.x"/>
+        <state_interface name="force.y"/>
+        <state_interface name="force.z"/>
+        <state_interface name="torque.x"/>
+        <state_interface name="torque.y"/>
         <state_interface name="torque.z"/>
         <param name="frame_id">tool_link</param>
         <param name="fx_range">100</param>
+        <param name="fy_range">100</param>
+        <param name="fz_range">100</param>
+        <param name="tx_range">15</param>
+        <param name="ty_range">15</param>
         <param name="tz_range">15</param>
       </sensor>

File: ros2_control_demo_description/rrbot_description/ros2_control/rrbot_system_multi_interface.ros2_control.xacro (robot description, xacro)
@@ -17,5 +17,5 @@
           <xacro:unless value="${use_fake_hardware}">
             <plugin>ros2_control_demo_hardware/RRBotSystemMultiInterfaceHardware</plugin>
-            <param name="example_param_hw_start_duration_sec">2.0</param>
+            <param name="example_param_hw_start_duration_sec">0.0</param>
             <param name="example_param_hw_stop_duration_sec">3.0</param>
             <param name="example_param_hw_slowdown">${slowdown}</param>
@@ -23,5 +23,5 @@
         </hardware>
       </xacro:unless>
-      <joint name="joint1">
+      <joint name="${prefix}joint1">
         <command_interface name="position">
           <param name="min">-1</param>
@@ -40,5 +40,5 @@
         <state_interface name="acceleration"/>
       </joint>
-      <joint name="joint2">
+      <joint name="${prefix}joint2">
         <command_interface name="position">
           <param name="min">-1</param>

File: ros2_control_demo_description/rrbot_description/ros2_control/rrbot_system_position_only.ros2_control.xacro (robot description, xacro)
@@ -17,5 +17,5 @@
           <xacro:unless value="${use_fake_hardware}">
             <plugin>ros2_control_demo_hardware/RRBotSystemPositionOnlyHardware</plugin>
-            <param name="example_param_hw_start_duration_sec">2.0</param>
+            <param name="example_param_hw_start_duration_sec">0.0</param>
             <param name="example_param_hw_stop_duration_sec">3.0</param>
             <param name="example_param_hw_slowdown">${slowdown}</param>
@@ -23,5 +23,5 @@
         </hardware>
       </xacro:unless>
-      <joint name="joint1">
+      <joint name="${prefix}joint1">
         <command_interface name="position">
           <param name="min">-1</param>
@@ -30,5 +30,5 @@
         <state_interface name="position"/>
       </joint>
-      <joint name="joint2">
+      <joint name="${prefix}joint2">
         <command_interface name="position">
           <param name="min">-1</param>

File: ros2_control_demo_description/rrbot_description/urdf/rrbot_modular_actuators.urdf.xacro (robot description, xacro)
@@ -8,8 +8,6 @@
   <xacro:arg name="use_sim" default="false" />
   <!-- Enable setting arguments from the launch file -->
-  <xacro:arg name="use_fake_hardware" default="false" />
-  <xacro:arg name="fake_sensor_commands" default="false" />
   <xacro:arg name="prefix" default="" />
-  <xacro:arg name="slowdown" default="100.0" />
+  <xacro:arg name="slowdown" default="2.0" />
   <!-- Import RRBot macro -->
   <xacro:include filename="$(find rrbot_description)/urdf/rrbot_description.urdf.xacro" />
@@ -19,5 +17,5 @@
   <xacro:include filename="$(find rrbot_description)/gazebo/rrbot.materials.xacro" />
   <!-- Import RRBot ros2_control description -->
-  <xacro:include filename="$(find rrbot_description)/ros2_control/rrbot_system_multi_interface.ros2_control.xacro" />
+  <xacro:include filename="$(find rrbot_description)/ros2_control/rrbot_modular_actuators.ros2_control.xacro" />
   <!-- Used for fixing robot -->
   <link name="world"/>
@@ -29,8 +27,6 @@
   </xacro:rrbot>
   <xacro:rrbot_gazebo prefix="$(arg prefix)" />
-  <xacro:rrbot_system_multi_interface
-    name="RRBotSystemMultiInterface" prefix="$(arg prefix)"
-    use_fake_hardware="$(arg use_fake_hardware)"
-    fake_sensor_commands="$(arg fake_sensor_commands)"
+  <xacro:rrbot_modular_actuators
+    name="RRBotModularJoint" prefix="$(arg prefix)"
     slowdown="$(arg slowdown)" />
 </robot>

File: ros2_control_demo_description/rrbot_description/urdf/rrbot_system_with_external_sensor.urdf.xacro (robot description, xacro)
@@ -1,4 +1,4 @@
 <?xml version="1.0"?>
-<!-- Revolute-Revolute Manipulator -->
+<!-- Revolute-Revolute Manipulator with a 6D Force-Torque sensor -->
 <!--
 Copied and modified from ROS1 example -
@@ -8,16 +8,16 @@
   <xacro:arg name="use_sim" default="false" />
   <!-- Enable setting arguments from the launch file -->
-  <xacro:arg name="use_fake_hardware" default="false" />
+  <xacro:arg name="use_fake_hardware" default="true" />
   <xacro:arg name="fake_sensor_commands" default="false" />
   <xacro:arg name="prefix" default="" />
-  <xacro:arg name="slowdown" default="100.0" />
+  <xacro:arg name="slowdown" default="50.0" />
   <!-- Import RRBot macro -->
   <xacro:include filename="$(find rrbot_description)/urdf/rrbot_description.urdf.xacro" />
-  <!-- Import all Gazebo-customization elements, including Gazebo colors -->
-  <xacro:include filename="$(find rrbot_description)/gazebo/rrbot.gazebo.xacro" />
   <!-- Import Rviz colors -->
   <xacro:include filename="$(find rrbot_description)/gazebo/rrbot.materials.xacro" />
   <!-- Import RRBot ros2_control description -->
-  <xacro:include filename="$(find rrbot_description)/ros2_control/rrbot_system_multi_interface.ros2_control.xacro" />
+  <xacro:include filename="$(find rrbot_description)/ros2_control/rrbot_system_position_only.ros2_control.xacro" />
+  <!-- Import RRBot external Force Torque Sensor description -->
+  <xacro:include filename="$(find rrbot_description)/ros2_control/external_rrbot_force_torque_sensor.ros2_control.xacro" />
   <!-- Used for fixing robot -->
   <link name="world"/>
@@ -28,9 +28,12 @@
     <origin xyz="0 0 0" rpy="0 0 0" />
   </xacro:rrbot>
-  <xacro:rrbot_gazebo prefix="$(arg prefix)" />
-  <xacro:rrbot_system_multi_interface
-    name="RRBotSystemMultiInterface" prefix="$(arg prefix)"
+  <xacro:rrbot_system_position_only
+    name="RRBotSystemPositionOnly" prefix="$(arg prefix)"
     use_fake_hardware="$(arg use_fake_hardware)"
     fake_sensor_commands="$(arg fake_sensor_commands)"
     slowdown="$(arg slowdown)" />
+  <xacro:external_rrbot_force_torque_sensor
+    name="ExternalRRBotFTSensor" prefix="$(arg prefix)"
+    use_fake_hardware="$(arg use_fake_hardware)"
+    fake_sensor_commands="$(arg fake_sensor_commands)" />
 </robot>
